File: Hardware/panel.sch (EAGLE design)
At the start: 86 parts, among them Q1 BC817-40LT1SMD, Q10 BC807-16LT1SMD, Q11 BC807-16LT1SMD, Q12 BC807-16LT1SMD, Q13 BC817-40LT1SMD, Q14 BC817-40LT1SMD, Q15 BC817-40LT1SMD, Q16 BC817-40LT1SMD, Q17 BC817-40LT1SMD, Q18 BC817-40LT1SMD, Q19 BC817-40LT1SMD, Q2 BC817-40LT1SMD, Q3 BC817-40LT1SMD, Q4 BC817-40LT1SMD, Q5 BC817-40LT1SMD, Q6 BC807-16LT1SMD, Q7 BC807-16LT1SMD, Q8 BC807-16LT1SMD, Q9 BC807-16LT1SMD, U1 MC7805CDT, X1 B16B-PHDSS, X2 52746-20

Commit message: оставил только часть с индикатором и переразвел ее под макетную плату
Parts:
- removed C1: 10uF 16v, rcl:CPOL-EUCT3216
- removed C2: 0.33uF, rcl:CPOL-EUCT3216
- removed C3: 0.1uF, rcl:CPOL-EUCT3216
- removed LED1: red, led_user:LEDRED_3MM
- removed LED2, LED3, LED4, LED5, LED6: green, led_user:LEDGREEN_3MM
- removed PAD1: (no value), wirepad:1,6/0,8
- removed Q1, Q14, Q15, Q16, Q17, Q18, Q19, Q2, Q3, Q4, Q5: BC817-40LT1SMD, transistor-npn:BC817-40LT1SMD
- removed Q10, Q11, Q12, Q7, Q8, Q9: BC807-16LT1SMD, transistor-pnp_user:BC807-16LT1SMD
- removed R1, R10, R11, R12, R15, R18, R19, R21, R22, R24, R25, R27, R28, R30, R31, R33, R36, R38, R4, R40, R42, R44, R46, R5, R6, R7, R8, R9: 4.7k, rcl:R-EU_R0805
- removed R17, R20, R23, R26, R29, R32: 2.2k, rcl:R-EU_R0805
- removed R2: 51, rcl:R-EU_R0805
- removed R3: 15k, rcl:R-EU_R0805
- removed R37, R39, R41, R43, R45, R47: 800, rcl:R-EU_R0805
- removed S1, S2, S3, S4, S5: 7mm, switch_user:TL11057MM
- removed U$1: TSOP4838FLAT, tsop:TSOP4838FLAT
- removed U1: MC7805CDT, _hhn_78xx_79xx_NCV78xx_d2pak_dpak:MC7805CDT
- removed X1: B16B-PHDSS, con-JST PHD:B16B-PHDSS
- removed X2: 52746-20, con-molex_user:52746-20
- added +24, +5_BOARD, GND, LED_SIG, OUT: LSP10, solpad:LSP10
Connections:
- removed net ADJLED: Q18.E, R44.2, X1.12
- removed net ADJLED_SIG: LED2.A, Q9.C, X2-11.S
- removed net DOWNLED: Q17.E, R42.2, X1.11
- removed net DOWNLED_SIG: LED3.A, Q10.C, X2-12.S
- removed net FFSW: Q5.C, S5.0@A, S5.0@B, X1.6
- removed net FF_SIG: R12.2, X2-9.S
- removed net FNSW: Q4.C, S4.0@A, S4.0@B, X1.5
- removed net FN_SIG: R10.2, X2-8.S
- removed net IR: R3.1, U$1.OUT, X1.14
- removed net LASERSW: Q3.C, S3.1@A, S3.1@B, X1.4
- removed net LASER_SIG: R8.2, X2-7.S
- removed net N$1: Q1.B, R1.2, R4.1
- removed net N$11: Q14.B, R36.1, R37.2
- removed net N$12: Q7.B, R15.1, R18.1
- removed net N$13: LED6.C, R17.2
- removed net N$14: Q8.B, R19.1, R21.1
- removed net N$15: LED1.C, R20.2
- removed net N$16: Q9.B, R22.1, R24.1
- removed net N$17: LED2.C, R23.2
- removed net N$18: Q10.B, R25.1, R27.1
- removed net N$19: LED3.C, R26.2
- removed net N$2: C1.+, R2.1, R3.2, U$1.V+
- removed net N$20: Q11.B, R28.1, R30.1
- removed net N$21: LED4.C, R29.2
- removed net N$22: Q12.B, R31.1, R33.1
- removed net N$23: LED5.C, R32.2
- removed net N$25: Q14.C, R15.2
- removed net N$26: Q15.B, R38.1, R39.2
- removed net N$27: Q15.C, R31.2
- removed net N$28: Q16.B, R40.1, R41.2
- removed net N$29: Q16.C, R28.2
- removed net N$30: Q17.B, R42.1, R43.2
- removed net N$31: Q17.C, R25.2
- removed net N$32: Q18.B, R44.1, R45.2
- removed net N$33: Q18.C, R22.2
- removed net N$34: Q19.B, R46.1, R47.2
- removed net N$35: Q19.C, R19.2
- removed net N$4: Q2.B, R5.2, R6.1
- removed net N$5: Q3.B, R7.2, R8.1
- removed net N$6: Q4.B, R10.1, R9.2
- removed net N$7: Q5.B, R11.2, R12.1
- removed net PRW_SIG: R4.2, X2-5.S
- removed net PWRLED: Q19.E, R46.2, X1.13
- removed net PWRLED_SIG: LED1.A, Q8.C, X2-10.S
- removed net PWR_SW: Q1.C, S1.1@A, S1.1@B, X1.2
- removed net SETSW: Q2.C, S2.0@A, S2.0@B, X1.3
- removed net SET_SIG: R6.2, X2-6.S
- removed net UPLED: Q14.E, R36.2, X1.8
- removed net UPLED_SIG: LED6.A, Q7.C, X2-15.S
- removed net VOUT_SB: C3.+, PAD1.P, U1.VOUT
- removed net XLED: Q16.E, R40.2, X1.10
- removed net XLED_SIG: LED4.A, Q11.C, X2-13.S
- removed net YLED: Q15.E, R38.2, X1.9
- removed net YLED_SIG: LED5.A, Q12.C, X2-14.S
- net +24V: now also +24.MP; no longer C2.+, Q10.E, Q11.E, Q12.E, Q7.E, Q8.E, Q9.E, R18.2, R21.2, R24.2, R27.2, R30.2, R33.2, U1.VIN, X2-17.S, X2-18.S, X2-19.S, X2-20.S
- net +5V: now also +5_BOARD.MP; no longer R2.2, R37.1, R39.1, R41.1, R43.1, R45.1, R47.1, X1.1
- net GND: now also GND.MP; no longer C1.-, C2.-, C3.-, Q1.E, Q2.E, Q3.E, Q4.E, Q5.E, R1.1, R11.1, R17.1, R20.1, R23.1, R26.1, R29.1, R32.1, R5.1, R7.1, R9.1, S1.0@A, S1.0@B, S2.1@A, S2.1@B, S3.0@A, S3.0@B, S4.1@A, S4.1@B, S5.1@A, S5.1@B, U$1.GND, U1.GND, X1.15, X1.16, X2-1.S, X2-2.S, X2-3.S, X2-4.S
- net LVLED: now also LED_SIG.MP; no longer X1.7
- net LVLLED_SIG: now also OUT.MP; no longer X2-16.S
Other:
- moved on the sheet: LED7, Q13, Q6, R13, R14, R16, R34, R35
